Commit message: logs updated

File: source/bdx/bdx/assets/models/bdx/bdx.urdf (robot description, URDF)
Before this commit: robot bdx, 21 links, 20 joints
Links:
- link ear_left: geometry collision mesh filename=../../meshes/bdx/ear_left.stl scale=0.001 0.001 0.001; visual mesh filename=../../meshes/bdx/ear_left.stl scale=0.001 0.001 0.001
- link ear_right: geometry collision mesh filename=../../meshes/bdx/ear_right.stl scale=0.001 0.001 0.001; visual mesh filename=../../meshes/bdx/ear_right.stl scale=0.001 0.001 0.001
- link head_body_pitch: geometry collision mesh filename=../../meshes/bdx/head_body_pitch.stl scale=0.001 0.001 0.001; visual mesh filename=../../meshes/bdx/head_body_pitch.stl scale=0.001 0.001 0.001
- link head_body_roll: geometry collision mesh filename=../../meshes/bdx/head_body_roll.stl scale=0.001 0.001 0.001; visual mesh filename=../../meshes/bdx/head_body_roll.stl scale=0.001 0.001 0.001
- link head_body_yaw: geometry collision mesh filename=../../meshes/bdx/head_body_yaw.stl scale=0.001 0.001 0.001; visual mesh filename=../../meshes/bdx/head_body_yaw.stl scale=0.001 0.001 0.001
- link left_foot_link: geometry collision mesh filename=../../meshes/bdx/left_foot.stl scale=0.001 0.001 0.001; visual mesh filename=../../meshes/bdx/left_foot.stl scale=0.001 0.001 0.001
- link left_hip: geometry collision mesh filename=../../meshes/bdx/left_hip.stl scale=0.001 0.001 0.001; visual mesh filename=../../meshes/bdx/left_hip.stl scale=0.001 0.001 0.001
- link left_hip_rotation: geometry collision mesh filename=../../meshes/bdx/left_hip_rotation.stl scale=0.001 0.001 0.001; visual mesh filename=../../meshes/bdx/left_hip_rotation.stl scale=0.001 0.001 0.001
- link left_shin: geometry collision mesh filename=../../meshes/bdx/left_shin.stl scale=0.001 0.001 0.001; visual mesh filename=../../meshes/bdx/left_shin.stl scale=0.001 0.001 0.001
- link left_thigh: geometry collision mesh filename=../../meshes/bdx/left_thigh.stl scale=0.001 0.001 0.001; visual mesh filename=../../meshes/bdx/left_thigh.stl scale=0.001 0.001 0.001
- link neck: geometry collision mesh filename=../../meshes/bdx/neck.stl scale=0.001 0.001 0.001; visual mesh filename=../../meshes/bdx/neck.stl scale=0.001 0.001 0.001
- link pelvis: geometry collision mesh filename=../../meshes/bdx/pelvis.stl scale=0.001 0.001 0.001; visual mesh filename=../../meshes/bdx/pelvis.stl scale=0.001 0.001 0.001
- link right_foot_link: geometry collision mesh filename=../../meshes/bdx/right_foot.stl scale=0.001 0.001 0.001; visual mesh filename=../../meshes/bdx/right_foot.stl scale=0.001 0.001 0.001
- link right_hip: geometry collision mesh filename=../../meshes/bdx/right_hip.stl scale=0.001 0.001 0.001; visual mesh filename=../../meshes/bdx/right_hip.stl scale=0.001 0.001 0.001
- link right_hip_rotation: geometry collision mesh filename=../../meshes/bdx/right_hip_rotation.stl scale=0.001 0.001 0.001; visual mesh filename=../../meshes/bdx/right_hip_rotation.stl scale=0.001 0.001 0.001
- link right_shin: geometry collision mesh filename=../../meshes/bdx/right_shin.stl scale=0.001 0.001 0.001; visual mesh filename=../../meshes/bdx/right_shin.stl scale=0.001 0.001 0.001
- link right_thigh: geometry collision mesh filename=../../meshes/bdx/right_thigh.stl scale=0.001 0.001 0.001; visual mesh filename=../../meshes/bdx/right_thigh.stl scale=0.001 0.001 0.001
